Commit message: Corrected URDF and added cylinders for smoother driving. Can increase STL rez on generator for future versions.

File: stickbot_generated_urdf/urdf/stickbot.urdf (robot description, URDF)
Before this commit: robot StickBot_1, 44 links, 43 joints
Links:
- removed link DiffDriveBase/RearRight
- removed link HEBI_SIM/DiffDriveBase/RearRight/X8_3
- added link hebi_x8_16_16Z_54, mass 5.000268491400921; collision mesh filename=package://stickbot_generated_urdf/meshes/hebi_x8_16_3z_prt.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 scale=0.001 0.001 0.001; visual mesh filename=package://stickbot_generated_urdf/meshes/hebi_x8_16_3z_prt.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 scale=0.001 0.001 0.001
- link pp_2074_08_0: geometry collision cylinder length=0.0254 radius=0.1016; visual mesh filename=package://stickbot_generated_urdf/meshes/pp_2074_08_prt.stl scale=0.001 0.001 0.001
- link pp_2074_08_1: geometry collision cylinder length=0.0254 radius=0.1016; visual mesh filename=package://stickbot_generated_urdf/meshes/pp_2074_08_prt.stl scale=0.001 0.001 0.001
- link pp_2074_08_2: geometry collision cylinder length=0.0254 radius=0.1016; visual mesh filename=package://stickbot_generated_urdf/meshes/pp_2074_08_prt.stl scale=0.001 0.001 0.001
- link pp_2074_08_3: geometry collision cylinder length=0.0254 radius=0.1016; visual mesh filename=package://stickbot_generated_urdf/meshes/pp_2074_08_prt.stl scale=0.001 0.001 0.001
Joints:
- removed joint DiffDriveBase/FrontLeft/X8_16
- removed joint DiffDriveBase/FrontRight/X8_16
- removed joint DiffDriveBase/RearLeft/X8_16
- removed joint DiffDriveBase/RearRight
- removed joint HEBI_SIM_JOINT/DiffDriveBase/RearRight
- removed joint a_2043_01_2_to_DiffDriveBase/RearRight
- added joint DiffDriveBase/FrontLeft/X8_3: type revolute, parent hebi_x8_16_2Z_0, child pm_2155_01_0, origin xyz=-2.75851691508e-18 -1.73288773498e-16 0.04505 rpy=-7.49879891331e-33 1.18329135783e-30 3.14159265359, axis 6.12323399574e-17 6.12323399574e-17 1.0, limit lower=-2.14e9 upper=+2.14e9 effort=100 velocity=100
- added joint DiffDriveBase/FrontRight/X8_3: type revolute, parent hebi_x8_16_1Z_0, child pm_2155_01_3, origin xyz=-2.75851691508e-18 -3.11802263455e-17 0.04505 rpy=7.49879891331e-33 1.18329135783e-30 3.14159265359, axis 6.12323399574e-17 6.12323399574e-17 1.0, limit lower=-2.14e9 upper=+2.14e9 effort=100 velocity=100
- added joint DiffDriveBase/RearLeft/X8_3: type revolute, parent hebi_x8_16_16Z_0, child pm_2155_01_2, origin xyz=-2.75851691508e-18 1.10928320807e-16 0.04505 rpy=1.65817885443e-45 1.18329135783e-30 3.14159265359, axis 6.12323399574e-17 6.12323399574e-17 1.0, limit lower=-2.14e9 upper=+2.14e9 effort=100 velocity=100
- added joint DiffDriveBase/RearRight/X8_3: type revolute, parent hebi_x8_16_16Z_54, child pm_2155_01_1, origin xyz=-2.75851691508e-18 -3.11802263455e-17 0.04505 rpy=7.49879891331e-33 1.18329135783e-30 3.14159265359, axis 6.12323399574e-17 6.12323399574e-17 1.0, limit lower=-2.14e9 upper=+2.14e9 effort=100 velocity=100
- added joint a_2043_01_2_to_hebi_x8_16_16Z_54: type fixed, parent a_2043_01_2, child hebi_x8_16_16Z_54, origin xyz=-6.52063401807e-18 8.5557524961e-17 0.0047752 rpy=-1.49975978266e-32 -6.12323399574e-17 3.14159265359
